File: pcb/TLE5012B.sch (KiCad schematic (older format))
At the start: 14 parts, among them J1 Conn_02x6_Odd_Even, J2 Conn_01x4, U1 ME6211C33M5G-N, U2 TLE5012B

Commit message: pcb: Minor updates to pcb
Only have one CS pin header (ground the others).
Add additional ground vias around perimeter of board.
Update 100nF LCSC part number
Parts:
- C2: LCSC# C167641 -> C14663; MFG# VJ0603Y104JXACW1BC -> (none)
- U2: symbol TLE5012B-rescue:TLE5012B-Sensor_Magnetic -> TLE5012B-rescue:TLE5012B-Sensor_Magnetic-TLE5012B-rescue; LCSC# (none) -> C123083
Connections:
- wire segments 45 -> 46
